Commit message: add FIR filter in chanel 0 fix bug of saturation PWM output

File: model/cepheus.urdf (robot description, URDF)
Before this commit: robot cepheus_robot, 8 links, 7 joints
Joints:
- joint reaction_wheel_joint: limit lower=-10.57 upper=20.57 effort=10 velocity=200.5 -> (none); type revolute -> continuous

Commit message: preliminary tests

File: model/cepheus.urdf (robot description, URDF)
Before this commit: robot cepheus_robot, 8 links, 7 joints
Links:
- removed link base_link
- removed link front_mouse
- added link camera; visual box size=0.018 0.0254 0.01
- added link cepheus; visual cylinder length=0.37 radius=0.15
- link left_mouse: geometry visual box size=0.09 .05 .03
- link reaction_wheel: geometry visual cylinder length=0.03 radius=0.045
- link right_mouse: geometry visual box size=0.09 .05 .03
Joints:
- removed joint f_odom
- added joint camera_joint: type fixed, parent cepheus, child camera, origin xyz=0.434 0.02025 0.1495 rpy=0 1.570796 0
- joint j_T1: origin xyz=0.085 0.147224319 0.23 rpy=0 0 -0.52 -> xyz=-0.085 0.147224319 0.23 rpy=0 0 0.523598776; parent base_link -> cepheus
- joint j_T2: origin xyz=-0.17 0 0.23 rpy=0 0 1.57 -> xyz=0.17 0 0.23 rpy=0 0 -1.570796327; parent base_link -> cepheus
- joint j_T3: origin xyz=0.085 -0.147224319 0.23 rpy=0 0 -2.62 -> xyz=-0.085 -0.147224319 0.23 rpy=0 0 -0.523598776; parent base_link -> cepheus
- joint l_odom: origin xyz=-0.1 0.1 0 rpy=0 0 0 -> xyz=0 0.1 0 rpy=0 0 0; parent base_link -> cepheus
- joint r_odom: origin xyz=-0.1 -0.1 0 rpy=0 0 0 -> xyz=0 -0.1 0 rpy=0 0 0; parent base_link -> cepheus
- joint reaction_wheel_joint: origin xyz=0 0 0 rpy=0 0 0 -> xyz=0.07 0 0 rpy=0 0 0; parent base_link -> cepheus

Commit message: lot of

File: model/cepheus.urdf (robot description, URDF)
Before this commit: robot cepheus, 8 links, 7 joints
Links:
- removed link T1
- removed link T2
- removed link T3
- removed link left_mouse
- removed link right_mouse
- added link probe; visual cylinder length=0.0016 radius=0.046; visual cylinder length=0.09955 radius=0.002
- added link probe_ft_sensor; visual cylinder length=0.026 radius=0.04
- link camera: geometry visual box size=0.018 0.0254 0.01; visual cylinder length=0.003 radius=0.0055
- link cepheus: geometry visual box size=0.254 0.02 0.02; visual cylinder length=0.0037 radius=0.0015
- link reaction_wheel: geometry visual cylinder length=0.03 radius=0.055
Joints:
- removed joint j_T1
- removed joint j_T2
- removed joint j_T3
- removed joint l_odom
- removed joint r_odom
- added joint botasys_joint: type fixed, parent cepheus, child probe_ft_sensor, origin xyz=0.41945 0.0 0.1698 rpy=1.570796327 0 1.570796327
- added joint probe_joint: type fixed, parent cepheus, child probe, origin xyz=0.519 0.0 0.1698 rpy=0 0 0
- joint camera_joint: origin xyz=0.434 0.02025 0.1495 rpy=0 1.570796 0 -> xyz=0.44625 0.014 0.1698 rpy=0 1.570796327 0

Commit message: huge update

File: model/cepheus.urdf (robot description, URDF)
Before this commit: robot cepheus, 5 links, 4 joints
Links:
- removed link camera
- removed link probe
- removed link probe_ft_sensor
- added link left_arm, mass 0.07974; collision box size=0.13 0.02 0.02; visual mesh filename=package://cepheus_robot/meshes/left_arm.STL
- added link left_finger, mass 0.15; visual box size=0.09 .05 .03
- added link left_forearm, mass 0.06392; collision box size=0.13 0.025 0.025; visual mesh filename=package://cepheus_robot/meshes/left_forearm.STL
- added link left_grip, mass 0.03547; collision box size=0.085 0.07 0.05; visual mesh filename=package://cepheus_robot/meshes/left_grip.STL
- link cepheus: mass None -> 7.11891369052411; geometry collision cylinder length=0.43 radius=0.2; visual mesh filename=package://cepheus_robot/meshes/cepheus.STL
- link reaction_wheel: geometry visual mesh filename=package://cepheus_robot/meshes/reaction_wheel.STL
Joints:
- removed joint botasys_joint
- removed joint camera_joint
- removed joint probe_joint
- added joint left_elbow: type revolute, parent left_arm, child left_forearm, origin xyz=0.18120 -0.01176 -0.002 rpy=0 0 0, axis 0 0 1, limit lower=-3.14 upper=1.5 effort=2 velocity=20
- added joint left_finger_joint: type revolute, parent left_grip, child left_finger, origin xyz=0.15965 0.01176 -0.00838 rpy=0 0 0 , axis 0 0 1, limit lower=-1 upper=1.35 effort=1 velocity=10
- added joint left_shoulder: type revolute, parent cepheus, child left_arm, origin xyz=0.17271 0.091404 0.05875 rpy=0 0 0, axis 0 0 1, limit lower=-0.86 upper=2.54 effort=20 velocity=20
- added joint left_wrist: type revolute, parent left_forearm, child left_grip, origin xyz=0.15965 0.01176 -0.00838 rpy=0 0 0 , axis 0 0 1, limit lower=-1.570796327 upper=1.570796327 effort=1 velocity=10
- joint reaction_wheel_joint: origin xyz=0.07 0 0 rpy=0 0 0 -> xyz=0.065 0 0.03815 rpy=0 0 0
